File: PCB_Prototipo_Proyecto_Final.kicad_pcb (KiCad board)
At the start: 2 copper layers, 0 parts

Commit message: Inicio de trazado de PCB
Se empezaron a acomodar los footprints.
Parts:
- added ?: , , F.Cu at (297.2, 58.4)
- added ?: , , F.Cu at (287.2, 203.3)
- added ?: , , F.Cu at (142.2, 203.3)
- added C1: 1 nF, Capacitor_SMD:C_0805_2012Metric, F.Cu at (477.3, 103.4)
- added C10: 1 nF, Capacitor_SMD:C_0805_2012Metric, F.Cu at (280.2, 150.2)
- added C11: 1 nF, Capacitor_SMD:C_0805_2012Metric, F.Cu at (472.8, 103.4)
- added C12: 1 nF, Capacitor_SMD:C_0805_2012Metric, F.Cu at (159.7, 112.8)
- added C13: 100 nF, 50V, Capacitor_SMD:C_0805_2012Metric, F.Cu at (236.0, 200.5)
- added C14: 470 uF, 50V, UUG1H471MNQ6MS:CAPAE1710X1750N, F.Cu at (240.3, 182.2)
- added C15: 220 uF, 10V, TPSE227K010R0100:TPSE227K016R0100V, F.Cu at (234.8, 194.8)
- added C16: 100 nF, 50V, Capacitor_SMD:C_0805_2012Metric, F.Cu at (231.5, 199.2)
- added C17: 10 uF, 10V, Capacitor_SMD:C_0805_2012Metric, F.Cu at (271.2, 182.3)
- added C18: 10 uF, 10V, Capacitor_SMD:C_0805_2012Metric, F.Cu at (240.4, 199.2)
- added C19: 10 uF, 10V, Capacitor_SMD:C_0805_2012Metric, F.Cu at (179.2, 156.3)
- added C2: 1 nF, Capacitor_SMD:C_0805_2012Metric, F.Cu at (481.7, 103.4)
- added C20: 100 nF, 50V, Capacitor_SMD:C_0805_2012Metric, F.Cu at (179.2, 159.3)
- added C21: 10 uF, 10V, Capacitor_SMD:C_0805_2012Metric, F.Cu at (174.7, 159.3)
- added C22: 100 nF, 50V, Capacitor_SMD:C_0805_2012Metric, F.Cu at (174.7, 156.3)
- added C23: 10 uF, 10V, Capacitor_SMD:C_0805_2012Metric, F.Cu at (205.2, 108.3)
- added C24: 100 nF, 50V, Capacitor_SMD:C_0805_2012Metric, F.Cu at (209.2, 108.3)
- added C3: 1 nF, Capacitor_SMD:C_0805_2012Metric, F.Cu at (472.8, 112.4)
- added C4: 1 nF, Capacitor_SMD:C_0805_2012Metric, F.Cu at (477.3, 106.4)
- added C5: 1 nF, Capacitor_SMD:C_0805_2012Metric, F.Cu at (486.2, 103.4)
- added C6: 1 nF, Capacitor_SMD:C_0805_2012Metric, F.Cu at (472.8, 115.4)
- added C7: 1 nF, Capacitor_SMD:C_0805_2012Metric, F.Cu at (280.2, 131.3)
- added C8: 1 nF, Capacitor_SMD:C_0805_2012Metric, F.Cu at (477.3, 112.4)
- added C9: 1 nF, Capacitor_SMD:C_0805_2012Metric, F.Cu at (477.3, 109.4)
- added D1: PMEG060V050EPD, Package_TO_SOT_SMD:Nexperia_CFP15_SOT-1289, F.Cu at (243.9, 194.8)
- added D2: FM4003-W, FM4003W:DIOM5025X231N, F.Cu at (222.0, 88.7)
- added D3: FM4003-W, FM4003W:DIOM5025X231N, F.Cu at (282.4, 89.1)
- added D4: FM4003-W, FM4003W:DIOM5025X231N, F.Cu at (162.1, 88.3)
- added D5: FM4003-W, FM4003W:DIOM5025X231N, F.Cu at (242.5, 89.4)
- added D6: FM4003-W, FM4003W:DIOM5025X231N, F.Cu at (182.2, 88.3)
- added D7: FM4003-W, FM4003W:DIOM5025X231N, F.Cu at (201.7, 88.4)
- added D8: FM4003-W, FM4003W:DIOM5025X231N, F.Cu at (262.5, 89.8)
- added IC1: MCP6486T-E_OT, MCP6486T-E_OT:MCP6486RT-E&slash_OT, F.Cu at (168.7, 112.8)
- added J1: VIN, TB002-500-02BE:TB00250002BE, F.Cu at (286.5, 188.8)
- added J10: Terminal_Sensores_Nivel, TB002-500-15BE:CUI_TB002-500-15BE, F.Cu at (316.8, 22.3)
- added J11: Terminal_Sensor_Flujo, TB002-500-03BE:SHDR3W100P0X500_1X3_1500X760X1000P, F.Cu at (373.0, 32.4)
- added J12: Rele_4, TB002-500-02BE:TB00250002BE, F.Cu at (220.8, 58.0)
- added J13: Rele_7, TB002-500-02BE:TB00250002BE, F.Cu at (281.0, 58.0)
- added J14: Rele_1, TB002-500-02BE:TB00250002BE, F.Cu at (160.7, 58.0)
- added J15: Rele_5, TB002-500-02BE:TB00250002BE, F.Cu at (240.9, 58.0)
- added J16: Rele_2, TB002-500-02BE:TB00250002BE, F.Cu at (180.7, 58.0)
- added J17: Rele_3, TB002-500-02BE:TB00250002BE, F.Cu at (200.8, 58.0)
- added J18: Rele_6, TB002-500-02BE:TB00250002BE, F.Cu at (260.9, 58.0)
- added J2: Conn_01x15, Connector_PinHeader_2.54mm:PinHeader_1x15_P2.54mm_Vertical, F.Cu at (206.2, 124.3)
- added J3: Conn_01x15, Connector_PinHeader_2.54mm:PinHeader_1x15_P2.54mm_Vertical, F.Cu at (232.2, 124.3)
- added J4: Terminal_Sensor_pH, TB001-500-04BE:TB00150004BE, F.Cu at (146.7, 101.8)
- added J5: Terminal_Sensor_Temp_Sumerg, TB002-500-03BE:SHDR3W100P0X500_1X3_1500X760X1000P, F.Cu at (356.4, 41.6)
- added J6: Terminal_Sensor_TDS, TB002-500-03BE:SHDR3W100P0X500_1X3_1500X760X1000P, F.Cu at (373.0, 41.6)
- added J7: Terminal_Sensor_Temp_Sumerg, TB002-500-03BE:SHDR3W100P0X500_1X3_1500X760X1000P, F.Cu at (295.5, 136.3)
- added J8: Terminal_Sensor_Iluminacion, TB002-500-03BE:SHDR3W100P0X500_1X3_1500X760X1000P, F.Cu at (339.9, 41.6)
- added J9: Terminal_Sensor_Temp_y_Hum, TB002-500-03BE:SHDR3W100P0X500_1X3_1500X760X1000P, F.Cu at (294.7, 145.3)
- added K1: SRD-05VDC-SL-C, SRD-05VDC-SL-C-Version_2:RELAY_SRD-05VDC-SL-C, F.Cu at (218.4, 75.2)
- added K2: SRD-05VDC-SL-C, SRD-05VDC-SL-C-Version_2:RELAY_SRD-05VDC-SL-C, F.Cu at (278.9, 74.9)
- added K3: SRD-05VDC-SL-C, SRD-05VDC-SL-C-Version_2:RELAY_SRD-05VDC-SL-C, F.Cu at (158.2, 75.3)
- added K4: SRD-05VDC-SL-C, SRD-05VDC-SL-C-Version_2:RELAY_SRD-05VDC-SL-C, F.Cu at (238.6, 75.1)
- added K5: SRD-05VDC-SL-C, SRD-05VDC-SL-C-Version_2:RELAY_SRD-05VDC-SL-C, F.Cu at (178.2, 75.3)
- added K6: SRD-05VDC-SL-C, SRD-05VDC-SL-C-Version_2:RELAY_SRD-05VDC-SL-C, F.Cu at (198.0, 75.3)
- added K7: SRD-05VDC-SL-C, SRD-05VDC-SL-C-Version_2:RELAY_SRD-05VDC-SL-C, F.Cu at (258.9, 75.1)
- added L1: 47 uH, 7447709470:WE-PD_1260_1245_1280_121054, F.Cu at (258.8, 191.9)
- added Q1: PMBT3904,235, PMBT3904,235:SOT95P230X110-3N, F.Cu at (213.5, 88.7)
- added Q2: PMBT3904,235, PMBT3904,235:SOT95P230X110-3N, F.Cu at (274.2, 89.5)
- added Q3: PMBT3904,235, PMBT3904,235:SOT95P230X110-3N, F.Cu at (152.2, 88.3)
- added Q4: PMBT3904,235, PMBT3904,235:SOT95P230X110-3N, F.Cu at (233.6, 89.3)
- added Q5: PMBT3904,235, PMBT3904,235:SOT95P230X110-3N, F.Cu at (172.2, 88.3)
- added Q6: PMBT3904,235, PMBT3904,235:SOT95P230X110-3N, F.Cu at (192.6, 88.6)
- added Q7: PMBT3904,235, PMBT3904,235:SOT95P230X110-3N, F.Cu at (254.3, 89.8)
- added R1: 549, 1/4W, Resistor_SMD:R_0805_2012Metric, F.Cu at (174.2, 112.7)
- added R10: 27, 1/2W, Resistor_SMD:R_0805_2012Metric, F.Cu at (495.0, 106.3)
- added R11: 27, 1/2W, Resistor_SMD:R_0805_2012Metric, F.Cu at (481.7, 115.3)
- added R12: 27, 1/2W, Resistor_SMD:R_0805_2012Metric, F.Cu at (481.7, 118.2)
- added R13: 27, 1/2W, Resistor_SMD:R_0805_2012Metric, F.Cu at (477.2, 118.3)
- added R14: 27, 1/2W, Resistor_SMD:R_0805_2012Metric, F.Cu at (477.2, 115.4)
- added R15: 27, 1/2W, Resistor_SMD:R_0805_2012Metric, F.Cu at (481.7, 109.4)
- added R16: 27, 1/2W, Resistor_SMD:R_0805_2012Metric, F.Cu at (472.8, 118.4)
- added R17: 27, 1/2W, Resistor_SMD:R_0805_2012Metric, F.Cu at (284.2, 131.2)
- added R18: 27, 1/2W, Resistor_SMD:R_0805_2012Metric, F.Cu at (276.2, 131.2)
- added R19: 27, 1/2W, Resistor_SMD:R_0805_2012Metric, F.Cu at (472.8, 121.3)
- added R2: 1K, 1/2W, Resistor_SMD:R_0805_2012Metric, F.Cu at (163.2, 112.8)
- added R20: 27, 1/2W, Resistor_SMD:R_0805_2012Metric, F.Cu at (495.0, 103.3)
- added R21: 27, 1/2W, Resistor_SMD:R_0805_2012Metric, F.Cu at (284.2, 150.3)
- added R22: 27, 1/2W, Resistor_SMD:R_0805_2012Metric, F.Cu at (276.2, 150.3)
- added R23: 27, 1/2W, Resistor_SMD:R_0805_2012Metric, F.Cu at (486.1, 112.3)
- added R24: 27, 1/2W, Resistor_SMD:R_0805_2012Metric, F.Cu at (155.7, 111.8)
- added R25: 820, 1/2W, Resistor_SMD:R_0805_2012Metric, F.Cu at (213.4, 93.3)
- added R26: 820, 1/2W, Resistor_SMD:R_0805_2012Metric, F.Cu at (274.1, 94.4)
- added R27: 820, 1/2W, Resistor_SMD:R_0805_2012Metric, F.Cu at (152.1, 93.3)
- added R28: 820, 1/2W, Resistor_SMD:R_0805_2012Metric, F.Cu at (233.6, 93.7)
- added R29: 820, 1/2W, Resistor_SMD:R_0805_2012Metric, F.Cu at (172.2, 93.3)
- added R3: 1K, 1/2W, Resistor_SMD:R_0805_2012Metric, F.Cu at (177.7, 112.9)
- added R30: 4.7K, 1/2W, Resistor_SMD:R_0805_2012Metric, F.Cu at (229.2, 108.3)
- added R31: 4.7K, 1/2W, Resistor_SMD:R_0805_2012Metric, F.Cu at (225.2, 108.3)
- added R32: 820, 1/2W, Resistor_SMD:R_0805_2012Metric, F.Cu at (192.5, 93.8)
- added R33: 820, 1/2W, Resistor_SMD:R_0805_2012Metric, F.Cu at (254.0, 94.5)
- added R4: 4,7K, 1/2W, Resistor_SMD:R_0805_2012Metric, F.Cu at (288.2, 131.2)
- added R5: 4,7K, 1/2W, Resistor_SMD:R_0805_2012Metric, F.Cu at (288.2, 150.4)
- added R6: 27, 1/2W, Resistor_SMD:R_0805_2012Metric, F.Cu at (472.8, 127.2)
- added R7: 27, 1/2W, Resistor_SMD:R_0805_2012Metric, F.Cu at (486.1, 106.4)
- added R8: 27, 1/2W, Resistor_SMD:R_0805_2012Metric, F.Cu at (472.8, 124.3)
- added R9: 27, 1/2W, Resistor_SMD:R_0805_2012Metric, F.Cu at (481.7, 112.3)
- added REF**: MountingHole_3.5mm_Pad, MountingHole:MountingHole_3.5mm_Pad, F.Cu at (142.2, 58.3)
- added U1: LM2596S-5, Package_TO_SOT_SMD:TO-263-5_TabPin3, F.Cu at (260.1, 178.7)
- added U2: LM1117-3.3, LM1117MPX-33NOPB:SOT230P700X180-4N, F.Cu at (273.7, 176.7)
- added U3: NXB0108PW-Q100J, Package_SO:TSSOP-20_4.4x6.5mm_P0.65mm, F.Cu at (187.2, 137.8)
- added U4: MCP23008-xSS, Package_SO:SSOP-20_5.3x7.2mm_P0.65mm, F.Cu at (217.2, 108.3)
Other:
- board outline added: 165.1 x 154.9 mm
