File: Entradas.kicad_sch (KiCad schematic)
At the start: 16 parts, among them IC1 UA741CP, J10 Terminal_Sensores_Nivel, J11 Terminal_Sensor_Flujo, J24 Pin GND, J4 Terminal_Sensor_pH, J5 Terminal_Sensor_CO2, J6 Terminal_Sensor_TDS, J7 Terminal_Sensor_Temp_Sumerg, J8 Terminal_Sensor_Iluminacion, J9 Terminal_Sensor_Temp_y_Hum

Commit message: Inicio de rerouteo.
Connections:
- net +3,3V: now also J9.3 (Pin_3); no longer J9.1 (Pin_1)
- net +5V: now also J10.12 (Pin_12), J10.15 (Pin_15), J10.3 (Pin_3), J10.6 (Pin_6), J10.9 (Pin_9); no longer J10.1 (Pin_1), J10.10 (Pin_10), J10.13 (Pin_13), J10.4 (Pin_4), J10.7 (Pin_7)
- net GND: now also J10.1 (Pin_1), J10.10 (Pin_10), J10.13 (Pin_13), J10.4 (Pin_4), J10.7 (Pin_7), J9.1 (Pin_1); no longer J10.12 (Pin_12), J10.15 (Pin_15), J10.3 (Pin_3), J10.6 (Pin_6), J10.9 (Pin_9), J9.3 (Pin_3)
- net SensorNivel_1: now also J10.14 (Pin_14); no longer J10.2 (Pin_2)
- net SensorNivel_2: now also J10.11 (Pin_11); no longer J10.5 (Pin_5)
- net SensorNivel_4: now also J10.5 (Pin_5); no longer J10.11 (Pin_11)
- net SensorNivel_5: now also J10.2 (Pin_2); no longer J10.14 (Pin_14)
Other:
- moved on the sheet: R5
Changed lines of the file:
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@@
   (junction (at 257.683 46.99) (diameter 0) (color 0 0 0 0)
   )
+  (junction (at 259.715 145.415) (diameter 0) (color 0 0 0 0)
+  )
   (junction (at 257.683 59.69) (diameter 0) (color 0 0 0 0)
   )
   (junction (at 264.795 59.69) (diameter 0) (color 0 0 0 0)
-  )
-  (junction (at 259.715 130.175) (diameter 0) (color 0 0 0 0)
   )
   (junction (at 257.683 71.12) (diameter 0) (color 0 0 0 0)
@@
     (stroke (width 0) (type default) (color 0 0 0 0))
   )
-  (wire (pts (xy 259.715 130.175) (xy 259.715 128.27))
+  (wire (pts (xy 259.715 140.335) (xy 259.715 145.415))
     (stroke (width 0) (type default) (color 0 0 0 0))
   )
@@
     (stroke (width 0) (type default) (color 0 0 0 0))
   )
+  (wire (pts (xy 250.825 140.335) (xy 259.715 140.335))
+    (stroke (width 0) (type default) (color 0 0 0 0))
+  )
   (wire (pts (xy 57.785 50.165) (xy 40.64 50.165))
     (stroke (width 0) (type default) (color 0 0 0 0))
@@
     (stroke (width 0) (type default) (color 0 0 0 0))
   )
-  (wire (pts (xy 259.715 130.175) (xy 267.97 130.175))
-    (stroke (width 0) (type default) (color 0 0 0 0))
-  )
   (wire (pts (xy 215.265 137.16) (xy 205.74 137.16))
     (stroke (width 0) (type default) (color 0 0 0 0))
@@
     (stroke (width 0) (type default) (color 0 0 0 0))
   )
-  (wire (pts (xy 259.715 135.255) (xy 259.715 130.175))
-    (stroke (width 0) (type default) (color 0 0 0 0))
-  )
   (wire (pts (xy 57.785 33.02) (xy 37.465 33.02))
     (stroke (width 0) (type default) (color 0 0 0 0))
@@
     (stroke (width 0) (type default) (color 0 0 0 0))
   )
-  (wire (pts (xy 250.825 140.335) (xy 257.302 140.335))
-    (stroke (width 0) (type default) (color 0 0 0 0))
-  )
   (wire (pts (xy 60.325 137.795) (xy 65.659 137.795))
     (stroke (width 0) (type default) (color 0 0 0 0))
@@
     (stroke (width 0) (type default) (color 0 0 0 0))
   )
+  (wire (pts (xy 259.715 145.415) (xy 259.715 147.32))
+    (stroke (width 0) (type default) (color 0 0 0 0))
+  )
   (wire (pts (xy 132.715 60.325) (xy 128.905 60.325))
     (stroke (width 0) (type default) (color 0 0 0 0))
@@
   )
   (polyline (pts (xy 177.038 11.938) (xy 177.038 166.116))
+    (stroke (width 0) (type default) (color 0 0 0 0))
+  )
+  (wire (pts (xy 259.715 145.415) (xy 267.97 145.415))
     (stroke (width 0) (type default) (color 0 0 0 0))
   )
@@
   )
   (text "NOTA DE RECORDATORIO: EL TERMINAL DE GND DE\nJ8 DEBERÁ CONECTARSE CON UN CABLE AL GND DE\nLA ALIMENTACIÓN DE ENTRADA EN J1"
-    (at 193.04 161.29 0)
+    (at 192.405 177.8 0)
     (effects (font (size 2 2) (thickness 0.254) bold) (justify left bottom))
   )
@@
     (effects (font (size 1.27 1.27)) (justify left bottom))
   )
-  (label "SensorNivel_2" (at 71.755 140.335 180)
+  (label "SensorNivel_4" (at 71.755 140.335 180)
     (effects (font (size 1 1)) (justify right bottom))
   )
@@
     (effects (font (size 1.27 1.27)) (justify left bottom))
   )
-  (label "SensorNivel_1" (at 71.755 132.715 180)
+  (label "SensorNivel_5" (at 71.755 132.715 180)
     (effects (font (size 1 1)) (justify right bottom))
   )
@@
     (effects (font (size 1.27 1.27)) (justify left bottom))
   )
-  (label "SensorNivel_4" (at 71.755 155.575 180)
+  (label "SensorNivel_2" (at 71.755 155.575 180)
     (effects (font (size 1 1)) (justify right bottom))
   )
@@
     (effects (font (size 1.27 1.27)) (justify left bottom))
   )
-  (label "SensorNivel_5" (at 71.755 163.195 180)
+  (label "SensorNivel_1" (at 71.755 163.195 180)
     (effects (font (size 1 1)) (justify right bottom))
   )
@@
     (effects (font (size 1.27 1.27)) (justify right))
   )
-  (hierarchical_label "+3,3V" (shape input) (at 259.715 128.27 90)
-    (effects (font (size 1.27 1.27)) (justify left))
+  (hierarchical_label "+3,3V" (shape input) (at 259.715 147.32 270)
+    (effects (font (size 1.27 1.27)) (justify right))
   )
   (hierarchical_label "Ilum_Analog" (shape output) (at 132.715 57.785 0)
@@
     (effects (font (size 1.27 1.27)) (justify left))
   )
-  (hierarchical_label "GND" (shape input) (at 257.302 140.335 0)
-    (effects (font (size 1.27 1.27)) (justify left))
-  )
-  (hierarchical_label "+5V" (shape input) (at 65.659 160.655 0)
+  (hierarchical_label "GND" (shape input) (at 259.715 135.255 0)
+    (effects (font (size 1.27 1.27)) (justify left))
+  )
+  (hierarchical_label "GND" (shape input) (at 65.659 160.655 0)
     (effects (font (size 1.27 1.27)) (justify left))
   )
@@
     (effects (font (size 1.27 1.27)) (justify left))
   )
-  (hierarchical_label "GND" (shape input) (at 65.659 165.735 0)
+  (hierarchical_label "+5V" (shape input) (at 65.659 165.735 0)
     (effects (font (size 1.27 1.27)) (justify left))
   )
@@
     (effects (font (size 1.27 1.27)) (justify left))
   )
-  (hierarchical_label "+5V" (shape input) (at 65.659 137.795 0)
+  (hierarchical_label "GND" (shape input) (at 65.659 137.795 0)
     (effects (font (size 1.27 1.27)) (justify left))
   )
@@
     (effects (font (size 1.27 1.27)) (justify right))
   )
-  (hierarchical_label "+5V" (shape input) (at 65.659 153.035 0)
-    (effects (font (size 1.27 1.27)) (justify left))
-  )
-  (hierarchical_label "GND" (shape input) (at 65.659 150.495 0)
+  (hierarchical_label "GND" (shape input) (at 65.659 153.035 0)
+    (effects (font (size 1.27 1.27)) (justify left))
+  )
+  (hierarchical_label "+5V" (shape input) (at 65.659 150.495 0)
     (effects (font (size 1.27 1.27)) (justify left))
   )
@@
     (effects (font (size 1.27 1.27)) (justify left))
   )
-  (hierarchical_label "GND" (shape input) (at 65.659 158.115 0)
+  (hierarchical_label "+5V" (shape input) (at 65.659 158.115 0)
     (effects (font (size 1.27 1.27)) (justify left))
   )
@@
     (effects (font (size 1.27 1.27)) (justify left))
   )
-  (hierarchical_label "+5V" (shape input) (at 65.659 130.175 0)
-    (effects (font (size 1.27 1.27)) (justify left))
-  )
-  (hierarchical_label "GND" (shape input) (at 65.659 135.255 0)
-    (effects (font (size 1.27 1.27)) (justify left))
-  )
-  (hierarchical_label "GND" (shape input) (at 65.659 142.875 0)
+  (hierarchical_label "GND" (shape input) (at 65.659 130.175 0)
+    (effects (font (size 1.27 1.27)) (justify left))
+  )
+  (hierarchical_label "+5V" (shape input) (at 65.659 135.255 0)
+    (effects (font (size 1.27 1.27)) (justify left))
+  )
+  (hierarchical_label "+5V" (shape input) (at 65.659 142.875 0)
     (effects (font (size 1.27 1.27)) (justify left))
   )
@@
     (effects (font (size 1.27 1.27)) (justify left))
   )
-  (hierarchical_label "+5V" (shape input) (at 65.659 145.415 0)
+  (hierarchical_label "GND" (shape input) (at 65.659 145.415 0)
     (effects (font (size 1.27 1.27)) (justify left))
   )
@@
     (in_bom yes) (on_board yes)
     (property "Reference" "J9" (id 0) (at 245.745 143.51 0))
-    (property "Value" "Terminal_Sensor_Temp_y_Hum" (id 1) (at 245.745 146.05 0))
+    (property "Value" "Terminal_Sensor_Temp_y_Hum" (id 1) (at 245.745 131.445 0))
     (property "Footprint" "TB002-500-03BE:SHDR3W100P0X500_1X3_1500X760X1000P" (id 2) (at 245.745 137.795 0)
       (effects (font (size 1.27 1.27)) hide)
@@
     (pin "2")
   )
-  (symbol (lib_id "Device:R_US") (at 267.97 133.985 0) (unit 1)
+  (symbol (lib_id "Device:R_US") (at 267.97 141.605 180) (unit 1)
     (in_bom yes) (on_board yes) (fields_autoplaced)
-    (property "Reference" "R5" (id 0) (at 270.51 132.7149 0)
-      (effects (font (size 1.27 1.27)) (justify left))
-    )
-    (property "Value" "4,7K, 1/8W" (id 1) (at 270.51 135.2549 0)
-      (effects (font (size 1.27 1.27)) (justify left))
-    )
-    (property "Footprint" "Resistor_SMD:R_0805_2012Metric" (id 2) (at 268.986 134.239 90)
-      (effects (font (size 1.27 1.27)) hide)
-    )
-    (property "Datasheet" "~" (id 3) (at 267.97 133.985 0)
-      (effects (font (size 1.27 1.27)) hide)
-    )
+    (property "Reference" "R5" (id 0) (at 270.51 140.3349 0)
+      (effects (font (size 1.27 1.27)) (justify right))
+    )
+    (property "Value" "4,7K, 1/8W" (id 1) (at 270.51 142.8749 0)
+      (effects (font (size 1.27 1.27)) (justify right))
+    )
+    (property "Footprint" "Resistor_SMD:R_0805_2012Metric" (id 2) (at 266.954 141.351 90)
+      (effects (font (size 1.27 1.27)) hide)
+    )
+    (property "Datasheet" "~" (id 3) (at 267.97 141.605 0)
+      (effects (font (size 1.27 1.27)) hide)
+    )
