File: Entradas.kicad_sch (KiCad schematic)
At the start: 16 parts, among them IC1 UA741CP, J10 Terminal_Sensores_Nivel, J11 Terminal_Sensor_Flujo, J24 Pin GND, J4 Terminal_Sensor_pH, J5 Terminal_Sensor_CO2, J6 Terminal_Sensor_TDS, J7 Terminal_Sensor_Temp_Sumerg, J8 Terminal_Sensor_Iluminacion, J9 Terminal_Sensor_Temp_y_Hum

Commit message: Cambios modelos 3D.
Changed lines of the file:
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@@
   )
   (text "NOTA DE RECORDATORIO: EL TERMINAL DE GND DE\nJ8 DEBERÁ CONECTARSE CON UN CABLE AL GND DE\nLA ALIMENTACIÓN DE ENTRADA EN J1"
-    (at 192.405 177.8 0)
+    (at 325.12 178.435 0)
     (effects (font (size 2 2) (thickness 0.254) bold) (justify left bottom))
   )
