File: Interfaces_GPIO.kicad_sch (KiCad schematic)
At the start: 6 parts, among them J34 Pin GND, U3 MCP23008-xP

Commit message: Correccion footprints
Se realizo el cambio de algunas footprints segun los componentes disponibles, como los capacitores de 470 uF o la inductancia de la fte switching, y tambien se cambio el LM2596 por el modelo ADJ, con el agregado de un divisor resistivo.
Parts:
- C19: footprint Capacitor_SMD:C_0805_2012Metric -> Capacitor_THT:CP_Radial_D5.0mm_P2.00mm
Changed lines of the file:
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@@
     (property "Reference" "C19" (id 0) (at 162.3263 70.485 90))
     (property "Value" "10 uF, 50V" (id 1) (at 165.735 73.025 90))
-    (property "Footprint" "Capacitor_SMD:C_0805_2012Metric" (id 2) (at 166.3903 76.5048 0)
+    (property "Footprint" "Capacitor_THT:CP_Radial_D5.0mm_P2.00mm" (id 2) (at 166.3903 76.5048 0)
       (effects (font (size 1.27 1.27)) hide)
     )
